Commit message: 算法优化和urdf更新

File: curobo/content/assets/robot/lycus/lycus.urdf (robot description, URDF)
Before this commit: robot lycus, 38 links, 37 joints
Links:
- removed link AR5-5_08L-W4C1C9-ZY2_base
- removed link AR5-5_08L-W4C1C9-ZY2_flan_link
- removed link AR5-5_08L-W4C1C9-ZY2_link1
- removed link AR5-5_08L-W4C1C9-ZY2_link2
- removed link AR5-5_08L-W4C1C9-ZY2_link3
- removed link AR5-5_08L-W4C1C9-ZY2_link4
- removed link AR5-5_08L-W4C1C9-ZY2_link5
- removed link AR5-5_08L-W4C1C9-ZY2_link6
- removed link AR5-5_08L-W4C1C9-ZY2_link7
- removed link AR5-5_08R-W4C1C9-ZY2_base
- removed link AR5-5_08R-W4C1C9-ZY2_flan_link
- removed link AR5-5_08R-W4C1C9-ZY2_link1
- removed link AR5-5_08R-W4C1C9-ZY2_link2
- removed link AR5-5_08R-W4C1C9-ZY2_link3
- removed link AR5-5_08R-W4C1C9-ZY2_link4
- removed link AR5-5_08R-W4C1C9-ZY2_link5
- removed link AR5-5_08R-W4C1C9-ZY2_link6
- removed link AR5-5_08R-W4C1C9-ZY2_link7
- removed link HouyuyanL_link
- removed link HouyuyanR_link
- removed link Qianyuyan_link
- removed link Shuangmu_link
- added link AR5-5_08L-W4C1C5-ZY2_base; collision mesh filename=meshes/AR5-5_08L-W4C1C5-ZY2_base.stl scale=0.001 0.001 0.001; visual mesh filename=meshes/AR5-5_08L-W4C1C5-ZY2_base.stl scale=0.001 0.001 0.001
- added link AR5-5_08L-W4C1C5-ZY2_flan_link, mass 0
- added link AR5-5_08L-W4C1C5-ZY2_link1, mass 2.166; collision mesh filename=meshes/AR5-5_08L-W4C1C5-ZY2_link1.stl scale=0.001 0.001 0.001; visual mesh filename=meshes/AR5-5_08L-W4C1C5-ZY2_link1.stl scale=0.001 0.001 0.001
- added link AR5-5_08L-W4C1C5-ZY2_link2, mass 1.903; collision mesh filename=meshes/AR5-5_08L-W4C1C5-ZY2_link2.stl scale=0.001 0.001 0.001; visual mesh filename=meshes/AR5-5_08L-W4C1C5-ZY2_link2.stl scale=0.001 0.001 0.001
- added link AR5-5_08L-W4C1C5-ZY2_link3, mass 1.845; collision mesh filename=meshes/AR5-5_08L-W4C1C5-ZY2_link3.stl scale=0.001 0.001 0.001; visual mesh filename=meshes/AR5-5_08L-W4C1C5-ZY2_link3.stl scale=0.001 0.001 0.001
- added link AR5-5_08L-W4C1C5-ZY2_link4, mass 1.037; collision mesh filename=meshes/AR5-5_08L-W4C1C5-ZY2_link4.stl scale=0.001 0.001 0.001; visual mesh filename=meshes/AR5-5_08L-W4C1C5-ZY2_link4.stl scale=.001 0.001 0.001
- added link AR5-5_08L-W4C1C5-ZY2_link5, mass 1.279; collision mesh filename=meshes/AR5-5_08L-W4C1C5-ZY2_link5.stl scale=0.001 0.001 0.001; visual mesh filename=meshes/AR5-5_08L-W4C1C5-ZY2_link5.stl scale=0.001 0.001 0.001
- added link AR5-5_08L-W4C1C5-ZY2_link6, mass 0.906; collision mesh filename=meshes/AR5-5_08L-W4C1C5-ZY2_link6.stl scale=0.001 0.001 0.001; visual mesh filename=meshes/AR5-5_08L-W4C1C5-ZY2_link6.stl scale=0.001 0.001 0.001
- added link AR5-5_08L-W4C1C5-ZY2_link7, mass 0.33; collision mesh filename=meshes/AR5-5_08L-W4C1C5-ZY2_link7.stl scale=0.001 0.001 0.001; visual mesh filename=meshes/AR5-5_08L-W4C1C5-ZY2_link7.stl scale=0.001 0.001 0.001
- added link AR5-5_08R-W4C1C5-ZY2_base; collision mesh filename=meshes/AR5-5_08R-W4C1C5-ZY2_base.stl scale=0.001 0.001 0.001; visual mesh filename=meshes/AR5-5_08R-W4C1C5-ZY2_base.stl scale=0.001 0.001 0.001
- added link AR5-5_08R-W4C1C5-ZY2_flan_link, mass 0
- added link AR5-5_08R-W4C1C5-ZY2_link1, mass 2.166; collision mesh filename=meshes/AR5-5_08R-W4C1C5-ZY2_link1.stl scale=0.001 0.001 0.001; visual mesh filename=meshes/AR5-5_08R-W4C1C5-ZY2_link1.stl scale=0.001 0.001 0.001
- added link AR5-5_08R-W4C1C5-ZY2_link2, mass 1.903; collision mesh filename=meshes/AR5-5_08R-W4C1C5-ZY2_link2.stl scale=0.001 0.001 0.001; visual mesh filename=meshes/AR5-5_08R-W4C1C5-ZY2_link2.stl scale=0.001 0.001 0.001
- added link AR5-5_08R-W4C1C5-ZY2_link3, mass 1.845; collision mesh filename=meshes/AR5-5_08R-W4C1C5-ZY2_link3.stl scale=0.001 0.001 0.001; visual mesh filename=meshes/AR5-5_08R-W4C1C5-ZY2_link3.stl scale=0.001 0.001 0.001
- added link AR5-5_08R-W4C1C5-ZY2_link4, mass 1.037; collision mesh filename=meshes/AR5-5_08R-W4C1C5-ZY2_link4.stl scale=0.001 0.001 0.001; visual mesh filename=meshes/AR5-5_08R-W4C1C5-ZY2_link4.stl scale=.001 0.001 0.001
- added link AR5-5_08R-W4C1C5-ZY2_link5, mass 1.279; collision mesh filename=meshes/AR5-5_08R-W4C1C5-ZY2_link5.stl scale=0.001 0.001 0.001; visual mesh filename=meshes/AR5-5_08R-W4C1C5-ZY2_link5.stl scale=0.001 0.001 0.001
- added link AR5-5_08R-W4C1C5-ZY2_link6, mass 0.906; collision mesh filename=meshes/AR5-5_08R-W4C1C5-ZY2_link6.stl scale=0.001 0.001 0.001; visual mesh filename=meshes/AR5-5_08R-W4C1C5-ZY2_link6.stl scale=0.001 0.001 0.001
- added link AR5-5_08R-W4C1C5-ZY2_link7, mass 0.33; collision mesh filename=meshes/AR5-5_08R-W4C1C5-ZY2_link7.stl scale=0.001 0.001 0.001; visual mesh filename=meshes/AR5-5_08R-W4C1C5-ZY2_link7.stl scale=0.001 0.001 0.001
- added link ChestRGBD_link, mass 0.02419; collision mesh filename=meshes/ChestRGBD_link.STL; visual mesh filename=meshes/ChestRGBD_link.STL
- added link HeadRGBD_link, mass 0.02419; collision mesh filename=meshes/HeadRGBD_link.STL; visual mesh filename=meshes/HeadRGBD_link.STL
- added link RGB1_link, mass 0.044686; collision mesh filename=meshes/RGB1_link.STL; visual mesh filename=meshes/RGB1_link.STL
- added link RGB2_link, mass 0.044686; collision mesh filename=meshes/RGB2_link.STL; visual mesh filename=meshes/RGB2_link.STL
- added link RGB3_link, mass 0.044686; collision mesh filename=meshes/RGB3_link.STL; visual mesh filename=meshes/RGB3_link.STL
- link Calf_link: mass 22.687 -> 5.9893
- link Chassis_link: mass 95.892 -> 83.6
- link Chest_link: mass 6.6409 -> 7.3291
- link Head_link: mass 1.4249 -> 0.72296
- link Neck_link: mass 0.81308 -> 0.61661
- link Thigh_link: mass 11.315 -> 12.921
- link Waist_link: mass 4.08058055678825 -> 15.046
- link Wheel1_link: mass 143.7 -> 3.2525
- link Wheel2_link: mass 143.7 -> 3.2525
- link Wheel3_link: mass 143.7 -> 3.2525
- link Wheel4_link: mass 143.7 -> 3.2525
Joints:
- removed joint AR5-5_08L-W4C1C9-ZY2_flan_joint
- removed joint AR5-5_08L-W4C1C9-ZY2_joint_1
- removed joint AR5-5_08L-W4C1C9-ZY2_joint_2
- removed joint AR5-5_08L-W4C1C9-ZY2_joint_3
- removed joint AR5-5_08L-W4C1C9-ZY2_joint_4
- removed joint AR5-5_08L-W4C1C9-ZY2_joint_5
- removed joint AR5-5_08L-W4C1C9-ZY2_joint_6
- removed joint AR5-5_08L-W4C1C9-ZY2_joint_7
- removed joint AR5-5_08R-W4C1C9-ZY2_flan_joint
- removed joint AR5-5_08R-W4C1C9-ZY2_joint_1
- removed joint AR5-5_08R-W4C1C9-ZY2_joint_2
- removed joint AR5-5_08R-W4C1C9-ZY2_joint_3
- removed joint AR5-5_08R-W4C1C9-ZY2_joint_4
- removed joint AR5-5_08R-W4C1C9-ZY2_joint_5
- removed joint AR5-5_08R-W4C1C9-ZY2_joint_6
- removed joint AR5-5_08R-W4C1C9-ZY2_joint_7
- removed joint Calf-joint
- removed joint Chest-joint
- removed joint Head-joint
- removed joint HouyuyanL_joint
- removed joint HouyuyanR_joint
- removed joint Neck-joint
- removed joint Qianyuyan_joint
- removed joint Shuangmu_joint
- removed joint Shuangmu_to_camera_joint
- removed joint Thigh-joint
- removed joint Waist-joint
- removed joint Whee1-joint
- removed joint Whee2-joint
- removed joint Whee3-joint
- removed joint Whee4-joint
- added joint AR5-5_08L-W4C1C5-ZY2_flan_joint: type fixed, parent AR5-5_08L-W4C1C5-ZY2_link7, child AR5-5_08L-W4C1C5-ZY2_flan_link, origin xyz=0 0 0.09 rpy=0 0 0
- added joint AR5-5_08L-W4C1C5-ZY2_joint_1: type revolute, parent AR5-5_08L-W4C1C5-ZY2_base, child AR5-5_08L-W4C1C5-ZY2_link1, origin xyz=0.0 0.0 0.0 rpy=0 0 0, axis 0 0 1, limit lower=-3.1067 upper=3.1067 effort=108 velocity=3.0543261909900763
- added joint AR5-5_08L-W4C1C5-ZY2_joint_2: type revolute, parent AR5-5_08L-W4C1C5-ZY2_link1, child AR5-5_08L-W4C1C5-ZY2_link2, origin xyz=0.0 0.0 0.1745 rpy=0 0 0, axis 0 1 0, limit lower=-2.0944 upper=2.0944 effort=108 velocity=3.0543261909900763
- added joint AR5-5_08L-W4C1C5-ZY2_joint_3: type revolute, parent AR5-5_08L-W4C1C5-ZY2_link2, child AR5-5_08L-W4C1C5-ZY2_link3, origin xyz=0.0 0.0 0.332 rpy=0 0 0, axis 0 0 1, limit lower=-3.1067 upper=3.1067 effort=66 velocity=4.71238898038469
- added joint AR5-5_08L-W4C1C5-ZY2_joint_4: type revolute, parent AR5-5_08L-W4C1C5-ZY2_link3, child AR5-5_08L-W4C1C5-ZY2_link4, origin xyz=0.0105 0.0 0.0 rpy=0 0 0, axis 0 1 0, limit lower=-1.0472 upper=2.5307 effort=66 velocity=5.235987755982989
- added joint AR5-5_08L-W4C1C5-ZY2_joint_5: type revolute, parent AR5-5_08L-W4C1C5-ZY2_link4, child AR5-5_08L-W4C1C5-ZY2_link5, origin xyz=-0.0105 0.0 0.278 rpy=0 0 0, axis 0 0 1, limit lower=-3.1067 upper=3.1067 effort=19 velocity=4.1887902047863905
- added joint AR5-5_08L-W4C1C5-ZY2_joint_6: type revolute, parent AR5-5_08L-W4C1C5-ZY2_link5, child AR5-5_08L-W4C1C5-ZY2_link6, origin xyz=0.0 0.0 0.0 rpy=0.0 0.0 0, axis 0 1 0, limit lower=-1.0472 upper=1.0472 effort=19 velocity=4.1887902047863905
- added joint AR5-5_08L-W4C1C5-ZY2_joint_7: type revolute, parent AR5-5_08L-W4C1C5-ZY2_link6, child AR5-5_08L-W4C1C5-ZY2_link7, origin xyz=0.0 0.0 0.0 rpy=0.0 0.0 0, axis 1 0 0, limit lower=-1.5708 upper=1.5708 effort=19 velocity=4.1887902047863905
- added joint AR5-5_08R-W4C1C5-ZY2_flan_joint: type fixed, parent AR5-5_08R-W4C1C5-ZY2_link7, child AR5-5_08R-W4C1C5-ZY2_flan_link, origin xyz=0 0 0.09 rpy=0 0 0
- added joint AR5-5_08R-W4C1C5-ZY2_joint_1: type revolute, parent AR5-5_08R-W4C1C5-ZY2_base, child AR5-5_08R-W4C1C5-ZY2_link1, origin xyz=0.0 0.0 0.0 rpy=0 0 0, axis 0 0 1, limit lower=-3.1067 upper=3.1067 effort=108 velocity=3.0543261909900763
- added joint AR5-5_08R-W4C1C5-ZY2_joint_2: type revolute, parent AR5-5_08R-W4C1C5-ZY2_link1, child AR5-5_08R-W4C1C5-ZY2_link2, origin xyz=0.0 0.0 0.1745 rpy=0 0 0, axis 0 1 0, limit lower=-2.0944 upper=2.0944 effort=108 velocity=3.0543261909900763
- added joint AR5-5_08R-W4C1C5-ZY2_joint_3: type revolute, parent AR5-5_08R-W4C1C5-ZY2_link2, child AR5-5_08R-W4C1C5-ZY2_link3, origin xyz=0.0 0.0 0.332 rpy=0 0 0, axis 0 0 1, limit lower=-3.1067 upper=3.1067 effort=66 velocity=4.71238898038469
- added joint AR5-5_08R-W4C1C5-ZY2_joint_4: type revolute, parent AR5-5_08R-W4C1C5-ZY2_link3, child AR5-5_08R-W4C1C5-ZY2_link4, origin xyz=0.0105 0.0 0.0 rpy=0 0 0, axis 0 1 0, limit lower=-1.0472 upper=2.5307 effort=66 velocity=5.235987755982989
- added joint AR5-5_08R-W4C1C5-ZY2_joint_5: type revolute, parent AR5-5_08R-W4C1C5-ZY2_link4, child AR5-5_08R-W4C1C5-ZY2_link5, origin xyz=-0.0105 0.0 0.278 rpy=0 0 0, axis 0 0 1, limit lower=-3.1067 upper=3.1067 effort=19 velocity=4.1887902047863905
- added joint AR5-5_08R-W4C1C5-ZY2_joint_6: type revolute, parent AR5-5_08R-W4C1C5-ZY2_link5, child AR5-5_08R-W4C1C5-ZY2_link6, origin xyz=0.0 0.0 0.0 rpy=0.0 0.0 0, axis 0 1 0, limit lower=-1.0472 upper=1.0472 effort=19 velocity=4.1887902047863905
- added joint AR5-5_08R-W4C1C5-ZY2_joint_7: type revolute, parent AR5-5_08R-W4C1C5-ZY2_link6, child AR5-5_08R-W4C1C5-ZY2_link7, origin xyz=0.0 0.0 0.0 rpy=0.0 0.0 0, axis 1 0 0, limit lower=-1.5708 upper=1.5708 effort=19 velocity=4.1887902047863905
- added joint Calf_joint: type revolute, parent Chassis_link, child Calf_link, origin xyz=0 0 0 rpy=0 0 0, axis 0 1 0, limit lower=-1.2217 upper=0.0873 effort=281 velocity=0.5236
- added joint ChestRGBD_joint: type fixed, parent Chest_link, child ChestRGBD_link, origin xyz=0.13803 0 0.0091575 rpy=0 0.34907 0, axis 0 0 0
- added joint Chest_joint: type revolute, parent Waist_link, child Chest_link, origin xyz=0 0 0.2705 rpy=0 0 0, axis 0 0 1, limit lower=-3.1416 upper=1.5708 effort=281 velocity=0.5236
- added joint HeadRGBD_joint: type fixed, parent Head_link, child HeadRGBD_link, origin xyz=0.086151 -0.033475 0.054122 rpy=0 0.35779 0, axis 0 0 0
- added joint Head_joint: type revolute, parent Neck_link, child Head_link, origin xyz=0.025 0.0331 0.2071 rpy=0 0 0, axis 0 1 0, limit lower=-0.5236 upper=0.6981 effort=8.9 velocity=0.5236
- added joint Neck_joint: type revolute, parent Chest_link, child Neck_link, origin xyz=-0.0025224 0 0.2298 rpy=0 0 0, axis 0 0 1, limit lower=-1.5708 upper=1.5708 effort=8.9 velocity=0.5236
- added joint RGB1_joint: type fixed, parent Head_link, child RGB1_link, origin xyz=0.10197 -0.033102 -0.044344 rpy=0 0 0, axis 0 0 0
- added joint RGB2_joint: type fixed, parent Head_link, child RGB2_link, origin xyz=-0.058272 0.035067 0.028914 rpy=0 0 2.1468, axis 0 0 0
- added joint RGB3_joint: type fixed, parent Head_link, child RGB3_link, origin xyz=-0.058272 -0.10127 0.028914 rpy=-0.00024534 0 -2.1468, axis 0 0 0
- added joint Thigh_joint: type revolute, parent Calf_link, child Thigh_link, origin xyz=0 0 0.35 rpy=0 0 0, axis 0 1 0, limit lower=-1.5708 upper=2.4435 effort=281 velocity=0.5236
- added joint Waist_joint: type revolute, parent Thigh_link, child Waist_link, origin xyz=0 0 0.48 rpy=0 0 0, axis 0 1 0, limit lower=-1.5708 upper=1.5708 effort=281 velocity=0.5236
- added joint Wheel1_joint: type revolute, parent Chassis_link, child Wheel1_link, origin xyz=0.18979 -0.172 -0.243 rpy=0 0 0, axis 0 1 0, limit lower=-6.28 upper=6.28 effort=50 velocity=6.28
- added joint Wheel2_joint: type revolute, parent Chassis_link, child Wheel2_link, origin xyz=0.18979 0.172 -0.243 rpy=0 0 0, axis 0 1 0, limit lower=-6.28 upper=6.28 effort=50 velocity=6.28
- added joint Wheel3_joint: type revolute, parent Chassis_link, child Wheel3_link, origin xyz=-0.31979 -0.172 -0.243 rpy=0 0 0, axis 0 1 0, limit lower=-6.28 upper=6.28 effort=50 velocity=6.28
- added joint Wheel4_joint: type revolute, parent Chassis_link, child Wheel4_link, origin xyz=-0.31979 0.172 -0.243 rpy=0 0 0, axis 0 1 0, limit lower=-6.28 upper=6.28 effort=50 velocity=6.28
- added joint head_rgbd_to_camera: type fixed, parent HeadRGBD_link, child camera_link, origin xyz=0 0 0 rpy=0 0 0
- joint left_arm_ee_joint: parent AR5-5_08L-W4C1C9-ZY2_flan_link -> AR5-5_08L-W4C1C5-ZY2_flan_link
- joint left_fixed: child AR5-5_08L-W4C1C9-ZY2_base -> AR5-5_08L-W4C1C5-ZY2_base; origin xyz=0.0 0.0775 0.1429 rpy=-1.57 1.57 0 -> xyz=-0.00109234234471721 0.0767398991492738 0.169871451048887 rpy=-1.4835273401367 0.00759597571992165 -0.0866018880051087
- joint right_arm_ee_joint: parent AR5-5_08R-W4C1C9-ZY2_flan_link -> AR5-5_08R-W4C1C5-ZY2_flan_link
- joint right_fixed: child AR5-5_08R-W4C1C9-ZY2_base -> AR5-5_08R-W4C1C5-ZY2_base; origin xyz=0.0 -0.0775 0.1429 rpy=1.57 1.57 0 -> xyz=-0.00109234234471728 -0.0767398991492542 0.169871451048887 rpy=1.48352734013671 0.00759597571992152 0.0866018880051084

Commit message: 更新lycus urdf和stl模型以及碰撞检测配置

File: curobo/content/assets/robot/lycus/lycus.urdf (robot description, URDF)
Before this commit: robot lycus, 39 links, 38 joints
Links:
- added link left_gripper_base, mass 1.5; collision mesh filename=meshes/gripper_drive_motor.stl; visual mesh filename=meshes/gripper_drive_motor.stl
- added link left_gripper_left_jaw, mass 0.37669144; collision mesh filename=meshes/gripper_left_finger.stl; visual mesh filename=meshes/gripper_left_finger.stl
- added link left_gripper_right_jaw, mass 0.37669236; collision mesh filename=meshes/gripper_right_finger.stl; visual mesh filename=meshes/gripper_right_finger.stl
- added link right_gripper_base, mass 1.5; collision mesh filename=meshes/gripper_drive_motor.stl; visual mesh filename=meshes/gripper_drive_motor.stl
- added link right_gripper_left_jaw, mass 0.37669144; collision mesh filename=meshes/gripper_left_finger.stl; visual mesh filename=meshes/gripper_left_finger.stl
- added link right_gripper_right_jaw, mass 0.37669236; collision mesh filename=meshes/gripper_right_finger.stl; visual mesh filename=meshes/gripper_right_finger.stl
Joints:
- added joint left_gripper: type prismatic, parent left_gripper_base, child left_gripper_right_jaw, origin xyz=0.01 0.1675 0.00072458 rpy=0 0 0, axis 1 0 0, limit lower=-0.042 upper=0 effort=10 velocity=3
- added joint left_gripper_mimic: type prismatic, parent left_gripper_base, child left_gripper_left_jaw, origin xyz=-0.01 0.1675 -0.02877542 rpy=0 0 0, axis 1 0 0, limit lower=0 upper=0.042 effort=10 velocity=3, mimic joint=left_gripper multiplier=-1 offset=0
- added joint left_gripper_mount: type fixed, parent AR5-5_08L-W4C1C5-ZY2_flan_link, child left_gripper_base, origin xyz=0 0 0 rpy=1.5707963267948966 0 3.141592653589793
- added joint right_gripper: type prismatic, parent right_gripper_base, child right_gripper_right_jaw, origin xyz=0.01 0.1675 0.00072458 rpy=0 0 0, axis 1 0 0, limit lower=-0.042 upper=0 effort=10 velocity=3
- added joint right_gripper_mimic: type prismatic, parent right_gripper_base, child right_gripper_left_jaw, origin xyz=-0.01 0.1675 -0.02877542 rpy=0 0 0, axis 1 0 0, limit lower=0 upper=0.042 effort=10 velocity=3, mimic joint=right_gripper multiplier=-1 offset=0
- added joint right_gripper_mount: type fixed, parent AR5-5_08R-W4C1C5-ZY2_flan_link, child right_gripper_base, origin xyz=0 0 0 rpy=1.5707963267948966 0 0
- joint left_arm_ee_joint: origin xyz=0 0 0 rpy=1.5707963267948966 0 0 -> xyz=0 0.2465 0.011975 rpy=0 0 0; parent AR5-5_08L-W4C1C5-ZY2_flan_link -> left_gripper_base
- joint right_arm_ee_joint: origin xyz=0 0 0 rpy=1.5707963267948966 0 0 -> xyz=0 0.2465 0.011975 rpy=0 0 0; parent AR5-5_08R-W4C1C5-ZY2_flan_link -> right_gripper_base

Commit message: 更新ee_link坐标系朝向

File: curobo/content/assets/robot/lycus/lycus.urdf (robot description, URDF)
Before this commit: robot lycus, 45 links, 44 joints
Joints:
- joint left_arm_ee_joint: origin xyz=0 0.2465 0.011975 rpy=0 0 0 -> xyz=0 0.2465 0.011975 rpy=0 -3.141592653589793 0
- joint right_arm_ee_joint: origin xyz=0 0.2465 0.011975 rpy=0 0 0 -> xyz=0 0.2465 0.011975 rpy=0 -3.141592653589793 0

Commit message: 修改夹爪角度

File: curobo/content/assets/robot/lycus/lycus.urdf (robot description, URDF)
Before this commit: robot lycus, 45 links, 44 joints
Joints:
- joint left_gripper_mount: origin xyz=0 0 0 rpy=1.5707963267948966 0 3.141592653589793 -> xyz=0 0 0 rpy=1.5707963267948966 0 4.71238898038469
- joint right_gripper_mount: origin xyz=0 0 0 rpy=1.5707963267948966 0 0 -> xyz=0 0 0 rpy=1.5707963267948966 0 -1.5707963267948966

Commit message: 统一 Lycus 相机连杆名称为 camera_01_link

File: curobo/content/assets/robot/lycus/lycus.urdf (robot description, URDF)
Before this commit: robot lycus, 45 links, 44 joints
Links:
- removed link camera_link
- added link camera_01_link
Joints:
- joint head_rgbd_to_camera: child camera_link -> camera_01_link
